File: BMS-Capstone/_autosave-Monitoring.kicad_sch (KiCad schematic)
At the start: 33 parts, among them IC1 BQ7694204PFBR

Commit message: Added PCB Design
Connections:
- net SPI_MISO: no longer IC1.28 (HDQ)
- new net SPI_MOSI: IC1.28 (HDQ)
Changed lines of the file:
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@@
 		)
 	)
-	(hierarchical_label "SPI_MISO"
+	(hierarchical_label "SPI_MOSI"
 		(shape input)
 		(at 162.56 105.41 0)
