File: BMS-Capstone/Monitoring.kicad_sch (KiCad schematic)
At the start: 33 parts, among them IC1 BQ7694204PFBR

Commit message: Ketchup
Connections:
- net SPI_MISO: no longer IC1.28 (HDQ)
- new net SPI_MOSI: IC1.28 (HDQ)
Other:
- moved on the sheet: C1, C10, C11, C12, C13, C14, C15, C16, C2, C3, C4, C5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

Commit message: im stupid
Parts:
- renumbered C9 to C, C16 to C, C14 to C, C8 to C, C10 to C, C1 to C, C11 to C, D1 to D, IC1 to IC, R13 to R, R9 to R, R12 to R, R1 to R
Changed lines of the file:
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@@
 		(dnp no)
 		(fields_autoplaced yes)
-		(property "Reference" "C9"
+		(property "Reference" "C"
 			(at 363.22 158.7499 0)
 			(effects
@@
 		(pin "2"
 		)
-		(instances
-			(project ""
-				(path "/f2da9442-ca05-4687-a880-d5cd24c39f1d/b0fa851b-ec8c-46af-afd4-efd0cc860c1e"
-					(reference "C9")
-					(unit 1)
-				)
-			)
-		)
+		(instances)
 	)
 	(symbol
@@
 		(dnp no)
 		(fields_autoplaced yes)
-		(property "Reference" "C16"
+		(property "Reference" "C"
 			(at 402.59 229.8699 0)
 			(effects
@@
 		(pin "2"
 		)
-		(instances
-			(project ""
-				(path "/f2da9442-ca05-4687-a880-d5cd24c39f1d/b0fa851b-ec8c-46af-afd4-efd0cc860c1e"
-					(reference "C16")
-					(unit 1)
-				)
-			)
-		)
+		(instances)
 	)
 	(symbol
@@
 		(on_board yes)
 		(dnp no)
-		(property "Reference" "IC1"
+		(property "Reference" "IC"
 			(at 397.51 159.258 0)
 			(effects
@@
 		(pin "31"
 		)
-		(instances
-			(project ""
-				(path "/f2da9442-ca05-4687-a880-d5cd24c39f1d/b0fa851b-ec8c-46af-afd4-efd0cc860c1e"
-					(reference "IC1")
-					(unit 1)
-				)
-			)
-		)
+		(instances)
 	)
 	(symbol
@@
 		(dnp no)
 		(fields_autoplaced yes)
-		(property "Reference" "#PWR06"
+		(property "Reference" "#PWR"
 			(at 398.78 243.84 0)
 			(effects
@@
 		(pin "1"
 		)
-		(instances
-			(project ""
-				(path "/f2da9442-ca05-4687-a880-d5cd24c39f1d/b0fa851b-ec8c-46af-afd4-efd0cc860c1e"
-					(reference "#PWR06")
-					(unit 1)
-				)
-			)
-		)
+		(instances)
 	)
 	(symbol
@@
 		(dnp no)
 		(fields_autoplaced yes)
-		(property "Reference" "R13"
+		(property "Reference" "R"
 			(at 386.08 262.8899 0)
 			(effects
@@
 		(pin "2"
 		)
-		(instances
-			(project ""
-				(path "/f2da9442-ca05-4687-a880-d5cd24c39f1d/b0fa851b-ec8c-46af-afd4-efd0cc860c1e"
-					(reference "R13")
-					(unit 1)
-				)
-			)
-		)
+		(instances)
 	)
 	(symbol
@@
 		(dnp no)
 		(fields_autoplaced yes)
-		(property "Reference" "#PWR05"
+		(property "Reference" "#PWR"
 			(at 394.97 292.1 0)
 			(effects
@@
 		(pin "1"
 		)
-		(instances
-			(project ""
-				(path "/f2da9442-ca05-4687-a880-d5cd24c39f1d/b0fa851b-ec8c-46af-afd4-efd0cc860c1e"
-					(reference "#PWR05")
-					(unit 1)
-				)
-			)
-		)
+		(instances)
 	)
 	(symbol
@@
 		(dnp no)
 		(fields_autoplaced yes)
-		(property "Reference" "R9"
+		(property "Reference" "R"
 			(at 341.63 148.59 90)
 			(effects
@@
 		(pin "1"
 		)
-		(instances
-			(project ""
-				(path "/f2da9442-ca05-4687-a880-d5cd24c39f1d/b0fa851b-ec8c-46af-afd4-efd0cc860c1e"
-					(reference "R9")
-					(unit 1)
-				)
-			)
-		)
+		(instances)
 	)
 	(symbol
@@
 		(dnp no)
 		(fields_autoplaced yes)
-		(property "Reference" "#PWR04"
+		(property "Reference" "#PWR"
 			(at 381 242.57 0)
 			(effects
@@
 		(pin "1"
 		)
-		(instances
-			(project ""
-				(path "/f2da9442-ca05-4687-a880-d5cd24c39f1d/b0fa851b-ec8c-46af-afd4-efd0cc860c1e"
-					(reference "#PWR04")
-					(unit 1)
-				)
-			)
-		)
+		(instances)
 	)
 	(symbol
@@
 		(dnp no)
 		(fields_autoplaced yes)
-		(property "Reference" "C14"
+		(property "Reference" "C"
 			(at 387.35 236.22 90)
 			(effects
@@
 		(pin "2"
 		)
-		(instances
-			(project ""
-				(path "/f2da9442-ca05-4687-a880-d5cd24c39f1d/b0fa851b-ec8c-46af-afd4-efd0cc860c1e"
-					(reference "C14")
-					(unit 1)
-				)
-			)
-		)
+		(instances)
 	)
 	(symbol
@@
 		(dnp no)
 		(fields_autoplaced yes)
-		(property "Reference" "C8"
+		(property "Reference" "C"
 			(at 354.33 158.7499 0)
 			(effects
@@
 		(pin "1"
 		)
-		(instances
-			(project ""
-				(path "/f2da9442-ca05-4687-a880-d5cd24c39f1d/b0fa851b-ec8c-46af-afd4-efd0cc860c1e"
-					(reference "C8")
-					(unit 1)
-				)
-			)
-		)
+		(instances)
 	)
 	(symbol
@@
 		(dnp no)
 		(fields_autoplaced yes)
-		(property "Reference" "#PWR01"
+		(property "Reference" "#PWR"
 			(at 350.52 170.18 0)
 			(effects
@@
 		(pin "1"
 		)
-		(instances
-			(project ""
-				(path "/f2da9442-ca05-4687-a880-d5cd24c39f1d/b0fa851b-ec8c-46af-afd4-efd0cc860c1e"
-					(reference "#PWR01")
-					(unit 1)
-				)
-			)
-		)
+		(instances)
 	)
 	(symbol
@@
 		(dnp no)
 		(fields_autoplaced yes)
-		(property "Reference" "R12"
+		(property "Reference" "R"
 			(at 387.35 271.78 90)
 			(effects
@@
 		(pin "1"
 		)
-		(instances
-			(project ""
-				(path "/f2da9442-ca05-4687-a880-d5cd24c39f1d/b0fa851b-ec8c-46af-afd4-efd0cc860c1e"
-					(reference "R12")
-					(unit 1)
-				)
-			)
-		)
+		(instances)
 	)
 	(symbol
@@
 		(dnp no)
 		(fields_autoplaced yes)
-		(property "Reference" "C10"
+		(property "Reference" "C"
 			(at 379.73 158.7499 0)
 			(effects
@@
 		(pin "1"
 		)
-		(instances
-			(project ""
-				(path "/f2da9442-ca05-4687-a880-d5cd24c39f1d/b0fa851b-ec8c-46af-afd4-efd0cc860c1e"
-					(reference "C10")
-					(unit 1)
-				)
-			)
-		)
+		(instances)
 	)
 	(symbol
@@
 		(dnp no)
 		(fields_autoplaced yes)
-		(property "Reference" "C1"
+		(property "Reference" "C"
 			(at 322.58 218.4399 0)
 			(effects
@@
 		(pin "2"
 		)
-		(instances
-			(project ""
-				(path "/f2da9442-ca05-4687-a880-d5cd24c39f1d/b0fa851b-ec8c-46af-afd4-efd0cc860c1e"
-					(reference "C1")
-					(unit 1)
-				)
-			)
-		)
+		(instances)
 	)
 	(symbol
@@
 		(on_board yes)
 		(dnp no)
-		(property "Reference" "R1"
+		(property "Reference" "R"
 			(at 308.61 165.354 90)
 			(effects
@@
 		(pin "2"
 		)
-		(instances
-			(project ""
-				(path "/f2da9442-ca05-4687-a880-d5cd24c39f1d/b0fa851b-ec8c-46af-afd4-efd0cc860c1e"
-					(reference "R1")
-					(unit 1)
-				)
-			)
-		)
+		(instances)
 	)
 	(symbol
@@
 		(dnp no)
 		(fields_autoplaced yes)
-		(property "Reference" "C11"
+		(property "Reference" "C"
 			(at 435.61 177.7999 0)
 			(effects
@@
 		(pin "1"
 		)
-		(instances
-			(project ""
-				(path "/f2da9442-ca05-4687-a880-d5cd24c39f1d/b0fa851b-ec8c-46af-afd4-efd0cc860c1e"
-					(reference "C11")
-					(unit 1)
-				)
-			)
-		)
+		(instances)
 	)
 	(symbol
@@
 		(dnp no)
 		(fields_autoplaced yes)
-		(property "Reference" "#PWR03"
+		(property "Reference" "#PWR"
 			(at 441.96 193.04 0)
 			(effects
@@
 		(pin "1"
 		)
-		(instances
-			(project ""
-				(path "/f2da9442-ca05-4687-a880-d5cd24c39f1d/b0fa851b-ec8c-46af-afd4-efd0cc860c1e"
-					(reference "#PWR03")
-					(unit 1)
-				)
-			)
-		)
+		(instances)
 	)
 	(symbol
@@
 		(dnp no)
 		(fields_autoplaced yes)
-		(property "Reference" "D1"
+		(property "Reference" "D"
 			(at 329.2475 148.59 0)
 			(effects
@@
 		(pin "2"
 		)
-		(instances
-			(project ""
-				(path "/f2da9442-ca05-4687-a880-d5cd24c39f1d/b0fa851b-ec8c-46af-afd4-efd0cc860c1e"
-					(reference "D1")
-					(unit 1)
-				)
-			)
-		)
-	)
-	(symbol
+		(instances)
+	)
+	(symbol

Commit message: did a thing
Parts:
- renumbered C to C?, D to D?, IC to IC?, R to R?
Changed lines of the file:
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@@
 		(dnp no)
 		(fields_autoplaced yes)
-		(property "Reference" "C"
+		(property "Reference" "C?"
 			(at 363.22 158.7499 0)
 			(effects
@@
 		(pin "2"
 		)
-		(instances)
+		(instances
+			(project "BMS"
+				(path "/f2da9442-ca05-4687-a880-d5cd24c39f1d/b0fa851b-ec8c-46af-afd4-efd0cc860c1e"
+					(reference "C?")
+					(unit 1)
+				)
+			)
+		)
 	)
 	(symbol
@@
 		(dnp no)
 		(fields_autoplaced yes)
-		(property "Reference" "C"
+		(property "Reference" "C?"
 			(at 402.59 229.8699 0)
 			(effects
@@
 		(pin "2"
 		)
-		(instances)
+		(instances
+			(project "BMS"
+				(path "/f2da9442-ca05-4687-a880-d5cd24c39f1d/b0fa851b-ec8c-46af-afd4-efd0cc860c1e"
+					(reference "C?")
+					(unit 1)
+				)
+			)
+		)
 	)
 	(symbol
@@
 		(on_board yes)
 		(dnp no)
-		(property "Reference" "IC"
+		(property "Reference" "IC?"
 			(at 397.51 159.258 0)
 			(effects
@@
 		(pin "31"
 		)
-		(instances)
+		(instances
+			(project "BMS"
+				(path "/f2da9442-ca05-4687-a880-d5cd24c39f1d/b0fa851b-ec8c-46af-afd4-efd0cc860c1e"
+					(reference "IC?")
+					(unit 1)
+				)
+			)
+		)
 	)
 	(symbol
@@
 		(dnp no)
 		(fields_autoplaced yes)
-		(property "Reference" "#PWR"
+		(property "Reference" "#PWR?"
 			(at 398.78 243.84 0)
 			(effects
@@
 		(pin "1"
 		)
-		(instances)
+		(instances
+			(project "BMS"
+				(path "/f2da9442-ca05-4687-a880-d5cd24c39f1d/b0fa851b-ec8c-46af-afd4-efd0cc860c1e"
+					(reference "#PWR?")
+					(unit 1)
+				)
+			)
+		)
 	)
 	(symbol
@@
 		(dnp no)
 		(fields_autoplaced yes)
-		(property "Reference" "R"
+		(property "Reference" "R?"
 			(at 386.08 262.8899 0)
 			(effects
@@
 		(pin "2"
 		)
-		(instances)
+		(instances
+			(project "BMS"
+				(path "/f2da9442-ca05-4687-a880-d5cd24c39f1d/b0fa851b-ec8c-46af-afd4-efd0cc860c1e"
+					(reference "R?")
+					(unit 1)
+				)
+			)
+		)
 	)
 	(symbol
@@
 		(dnp no)
 		(fields_autoplaced yes)
-		(property "Reference" "#PWR"
+		(property "Reference" "#PWR?"
 			(at 394.97 292.1 0)
 			(effects
@@
 		(pin "1"
 		)
-		(instances)
+		(instances
+			(project "BMS"
+				(path "/f2da9442-ca05-4687-a880-d5cd24c39f1d/b0fa851b-ec8c-46af-afd4-efd0cc860c1e"
+					(reference "#PWR?")
+					(unit 1)
+				)
+			)
+		)
 	)
 	(symbol
@@
 		(dnp no)
 		(fields_autoplaced yes)
-		(property "Reference" "R"
+		(property "Reference" "R?"
 			(at 341.63 148.59 90)
 			(effects
@@
 		(pin "1"
 		)
-		(instances)
+		(instances
+			(project "BMS"
+				(path "/f2da9442-ca05-4687-a880-d5cd24c39f1d/b0fa851b-ec8c-46af-afd4-efd0cc860c1e"
+					(reference "R?")
+					(unit 1)
+				)
+			)
+		)
 	)
 	(symbol
@@
 		(dnp no)
 		(fields_autoplaced yes)
-		(property "Reference" "#PWR"
+		(property "Reference" "#PWR?"
 			(at 381 242.57 0)
 			(effects
@@
 		(pin "1"
 		)
-		(instances)
+		(instances
+			(project "BMS"
+				(path "/f2da9442-ca05-4687-a880-d5cd24c39f1d/b0fa851b-ec8c-46af-afd4-efd0cc860c1e"
+					(reference "#PWR?")
+					(unit 1)
+				)
+			)
+		)
 	)
 	(symbol
@@
 		(dnp no)
 		(fields_autoplaced yes)
-		(property "Reference" "C"
+		(property "Reference" "C?"
 			(at 387.35 236.22 90)
 			(effects
@@
 		(pin "2"
 		)
-		(instances)
+		(instances
+			(project "BMS"
+				(path "/f2da9442-ca05-4687-a880-d5cd24c39f1d/b0fa851b-ec8c-46af-afd4-efd0cc860c1e"
+					(reference "C?")
+					(unit 1)
+				)
+			)
+		)
 	)
 	(symbol
@@
 		(dnp no)
 		(fields_autoplaced yes)
-		(property "Reference" "C"
+		(property "Reference" "C?"
 			(at 354.33 158.7499 0)
 			(effects
@@
 		(pin "1"
 		)
-		(instances)
+		(instances
+			(project "BMS"
+				(path "/f2da9442-ca05-4687-a880-d5cd24c39f1d/b0fa851b-ec8c-46af-afd4-efd0cc860c1e"
+					(reference "C?")
+					(unit 1)
+				)
+			)
+		)
 	)
 	(symbol
@@
 		(dnp no)
 		(fields_autoplaced yes)
-		(property "Reference" "#PWR"
+		(property "Reference" "#PWR?"
 			(at 350.52 170.18 0)
 			(effects
@@
 		(pin "1"
 		)
-		(instances)
+		(instances
+			(project "BMS"
+				(path "/f2da9442-ca05-4687-a880-d5cd24c39f1d/b0fa851b-ec8c-46af-afd4-efd0cc860c1e"
+					(reference "#PWR?")
+					(unit 1)
+				)
+			)
+		)
 	)
 	(symbol
@@
 		(dnp no)
 		(fields_autoplaced yes)
-		(property "Reference" "R"
+		(property "Reference" "R?"
 			(at 387.35 271.78 90)
 			(effects
@@
 		(pin "1"
 		)
-		(instances)
+		(instances
+			(project "BMS"
+				(path "/f2da9442-ca05-4687-a880-d5cd24c39f1d/b0fa851b-ec8c-46af-afd4-efd0cc860c1e"
+					(reference "R?")
+					(unit 1)
+				)
+			)
+		)
 	)
 	(symbol
@@
 		(dnp no)
 		(fields_autoplaced yes)
-		(property "Reference" "C"
+		(property "Reference" "C?"
 			(at 379.73 158.7499 0)
 			(effects
@@
 		(pin "1"
 		)
-		(instances)
+		(instances
+			(project "BMS"
+				(path "/f2da9442-ca05-4687-a880-d5cd24c39f1d/b0fa851b-ec8c-46af-afd4-efd0cc860c1e"
+					(reference "C?")
+					(unit 1)
+				)
+			)
+		)
 	)
 	(symbol
@@
 		(dnp no)
 		(fields_autoplaced yes)
-		(property "Reference" "C"
+		(property "Reference" "C?"
 			(at 322.58 218.4399 0)
 			(effects
@@
 		(pin "2"
 		)
-		(instances)
+		(instances
+			(project "BMS"
+				(path "/f2da9442-ca05-4687-a880-d5cd24c39f1d/b0fa851b-ec8c-46af-afd4-efd0cc860c1e"
+					(reference "C?")
+					(unit 1)
+				)
+			)
+		)
 	)
 	(symbol
@@
 		(on_board yes)
 		(dnp no)
-		(property "Reference" "R"
+		(property "Reference" "R?"
 			(at 308.61 165.354 90)
 			(effects
@@
 		(pin "2"
 		)
-		(instances)
+		(instances
+			(project "BMS"
+				(path "/f2da9442-ca05-4687-a880-d5cd24c39f1d/b0fa851b-ec8c-46af-afd4-efd0cc860c1e"
+					(reference "R?")
+					(unit 1)
+				)
+			)
+		)
 	)
 	(symbol
@@
 		(dnp no)
 		(fields_autoplaced yes)
-		(property "Reference" "C"
+		(property "Reference" "C?"
 			(at 435.61 177.7999 0)
 			(effects
@@
 		(pin "1"
 		)
-		(instances)
+		(instances
+			(project "BMS"
+				(path "/f2da9442-ca05-4687-a880-d5cd24c39f1d/b0fa851b-ec8c-46af-afd4-efd0cc860c1e"
+					(reference "C?")
+					(unit 1)
+				)
+			)
+		)
 	)
 	(symbol
@@
 		(dnp no)
 		(fields_autoplaced yes)
-		(property "Reference" "#PWR"
+		(property "Reference" "#PWR?"
 			(at 441.96 193.04 0)
 			(effects
@@
 		(pin "1"
 		)
-		(instances)
+		(instances
+			(project "BMS"
+				(path "/f2da9442-ca05-4687-a880-d5cd24c39f1d/b0fa851b-ec8c-46af-afd4-efd0cc860c1e"
+					(reference "#PWR?")
+					(unit 1)
+				)
+			)
+		)
 	)
 	(symbol
@@
 		(dnp no)
 		(fields_autoplaced yes)
-		(property "Reference" "D"
+		(property "Reference" "D?"
 			(at 329.2475 148.59 0)
 			(effects
@@
 		(pin "2"
 		)
-		(instances)
-	)
-	(symbol
+		(instances
+			(project "BMS"
+				(path "/f2da9442-ca05-4687-a880-d5cd24c39f1d/b0fa851b-ec8c-46af-afd4-efd0cc860c1e"
+					(reference "D?")
+					(unit 1)
+				)
+			)
+		)
+	)
+	(symbol
