File: BMS-Capstone/Monitoring.kicad_sch (KiCad schematic)
At the start: 0 parts

Commit message: Added main Schematic to branch and linked components to PCB
Parts:
- added C1, C2, C3, C4, C5, C6, C7: 220n, Capacitor_SMD:C_0805_2012Metric, symbol Device:C
- added C10: 0.47u, Capacitor_SMD:C_0805_2012Metric, symbol Device:C
- added C11, C12, C13: 22n, Capacitor_SMD:C_0805_2012Metric, symbol Device:C
- added C14, C15, C9: 100p, Capacitor_SMD:C_0805_2012Metric, symbol Device:C
- added C16: 2.2u, Capacitor_SMD:C_0805_2012Metric, symbol Device:C
- added C8: 1u, Capacitor_SMD:C_0805_2012Metric, symbol Device:C
- added D1, D2: D_Schottky, Diode_SMD:D_0805_2012Metric, symbol Device:D_Schottky
- added IC1: BQ7694204PFBR, Package_QFP:Texas_PHP0048E_HTQFP-48-1EP_7x7mm_P0.5mm_EP6.5x6.5mm_Mask3.62x3.62mm, symbol SamacSys_Parts:BQ7694204PFBR
- added R1, R2, R3, R4, R5, R6, R7, R8: 20, Resistor_SMD:R_0805_2012Metric, symbol Device:R
- added R10, R11: 150, Resistor_SMD:R_0805_2012Metric, symbol Device:R
- added R12: 0.001, Resistor_SMD:R_0805_2012Metric, symbol Device:R
- added R13, R14, R9: 100, Resistor_SMD:R_0805_2012Metric, symbol Device:R
Connections:
- new net: D2.1 (K), R10.1
- new net: C10.1, C8.1, C9.1, IC1.47 (BAT), R9.2
- new net: C16.1, IC1.24 (REG18)
- new net: C1.1, C2.2, IC1.15 (VC1), R7.2
- new net: C5.1, C6.2, IC1.10 (VC5), R3.2
- new net: C4.1, C5.2, IC1.12 (VC4), R4.2
- new net: C3.1, C4.2, IC1.13 (VC3), R5.2
- new net: C2.1, C3.2, IC1.14 (VC2), R6.2
- new net: C1.2, IC1.16 (VC0), R8.2
- new net: C14.2, C15.2, IC1.18 (SRP), R13.1
- new net: C14.1, C15.1, IC1.20 (SRN), R14.1
- new net: C11.1, IC1.36 (REGIN), R11.2
- new net: C10.2, IC1.46 (CP1)
- new net: C7.1, IC1.6 (VC7), R1.2
- new net: C6.1, C7.2, IC1.8 (VC6), R2.2
- new net: D1.1 (K), R9.1
- new net: R10.2, R11.1
- new net 1n: R12.1, R13.2, R8.1
- new net 1p: R7.1
- new net 2p: R6.1
- new net 3.3V: C13.1, IC1.34 (REG2)
- new net 3p: R5.1
- new net 4p: R4.1
- new net 5V: C12.1, IC1.35 (REG1)
- new net 5p: R3.1
- new net 6p: R2.1
- new net 7p: D1.2 (A), D2.2 (A), R1.1
- new net GND: C11.2, C12.2, C13.2, C16.2, C8.2, C9.2, IC1.17 (VSS), R12.2, R14.2
- new net INT: IC1.25 (ALERT)
- new net SPI_CS: IC1.29 (CFETOFF)
- new net SPI_MISO: IC1.27 (SDA)
- new net SPI_MOSI: IC1.28 (HDQ)
- new net SPI_SCLK: IC1.26 (SCL)
Other:
- note added: "NOTE: # = Cell number P/N = Positive / Negitive Terminal See Datasheet : https://drive.google.com/drive/u/1/folders/1Yq_641eaV3LJ5fxU185z7kZlac__CeCr"

Commit message: relinked footprints
Parts:
- renumbered C7 to C31, C5 to C32, C3 to C33, C1 to C34, C6 to C35, C4 to C36, C2 to C37, C8 to C38, C9 to C39, C10 to C40, C14 to C41, C15 to C42, C16 to C43, C12 to C44, C13 to C45, C11 to C46, D2 to D1, D1 to D2, IC1 to IC7, R1 to R44, R2 to R45, R3 to R46, R4 to R47, R5 to R48, R6 to R49, R7 to R50, R8 to R51, R9 to R52, R10 to R53, R11 to R54, R13 to R55, R12 to R56, R14 to R57
