File: BMS-Capstone/Monitoring.kicad_sch (KiCad schematic)
At the start: 33 parts, among them IC7 BQ7694204PFBR, J5 Conn_01x02_Socket

Commit message: routing for TI chip
Connections:
- net 1n: no longer J5.1 (Pin_1), R13M1.2
- new net: J5.1 (Pin_1), R13M1.2
Changed lines of the file:
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@@
 	)
 	(junction
-		(at 383.54 278.13)
-		(diameter 0)
-		(color 0 0 0 0)
-	)
-	(junction
 		(at 407.67 186.69)
 		(diameter 0)
@@
 	)
 	(junction
-		(at 300.99 223.52)
-		(diameter 0)
-		(color 0 0 0 0)
-	)
-	(junction
 		(at 318.77 200.66)
 		(diameter 0)
@@
 	)
 	(junction
+		(at 391.16 273.05)
+		(diameter 0)
+		(color 0 0 0 0)
+	)
+	(junction
 		(at 359.41 154.94)
 		(diameter 0)
@@
 	(wire
 		(pts
-			(xy 431.8 182.88) (xy 431.8 186.69)
+			(xy 419.1 243.84) (xy 438.15 243.84)
 		)
 		(stroke
@@
 	(wire
 		(pts
-			(xy 410.21 171.45) (xy 410.21 184.15)
+			(xy 431.8 182.88) (xy 431.8 186.69)
 		)
 		(stroke
@@
 	(wire
 		(pts
-			(xy 375.92 163.83) (xy 375.92 166.37)
+			(xy 410.21 171.45) (xy 410.21 184.15)
 		)
 		(stroke
@@
 	(wire
 		(pts
-			(xy 312.42 193.04) (xy 318.77 193.04)
+			(xy 375.92 163.83) (xy 375.92 166.37)
 		)
 		(stroke
@@
 	(wire
 		(pts
-			(xy 383.54 267.97) (xy 383.54 278.13)
+			(xy 312.42 193.04) (xy 318.77 193.04)
 		)
 		(stroke
@@
 	(wire
 		(pts
-			(xy 318.77 193.04) (xy 323.85 193.04)
+			(xy 383.54 267.97) (xy 383.54 278.13)
 		)
 		(stroke
@@
 	(wire
 		(pts
-			(xy 383.54 243.84) (xy 383.54 255.27)
+			(xy 318.77 193.04) (xy 323.85 193.04)
 		)
 		(stroke
@@
 	(wire
 		(pts
-			(xy 295.9642 223.52) (xy 300.99 223.52)
+			(xy 383.54 243.84) (xy 383.54 255.27)
 		)
 		(stroke
@@
 	(wire
 		(pts
+			(xy 391.16 273.05) (xy 419.1 273.05)
+		)
+		(stroke
+			(width 0)
+			(type default)
+		)
+	)
+	(wire
+		(pts
 			(xy 391.16 278.13) (xy 394.97 278.13)
 		)
@@
 	(wire
 		(pts
-			(xy 300.99 278.13) (xy 383.54 278.13)
+			(xy 391.16 233.68) (xy 391.16 243.84)
 		)
 		(stroke
@@
 	(wire
 		(pts
-			(xy 391.16 233.68) (xy 391.16 243.84)
+			(xy 344.17 142.24) (xy 332.74 142.24)
 		)
 		(stroke
@@
 	(wire
 		(pts
-			(xy 344.17 142.24) (xy 332.74 142.24)
+			(xy 383.54 278.13) (xy 386.08 278.13)
 		)
 		(stroke
@@
 	(wire
 		(pts
-			(xy 383.54 278.13) (xy 386.08 278.13)
+			(xy 323.85 208.28) (xy 335.2529 208.28)
 		)
 		(stroke
@@
 	(wire
 		(pts
-			(xy 323.85 208.28) (xy 335.2529 208.28)
+			(xy 351.79 194.31) (xy 363.22 194.31)
 		)
 		(stroke
@@
 	(wire
 		(pts
-			(xy 351.79 194.31) (xy 363.22 194.31)
+			(xy 419.1 273.05) (xy 419.1 243.84)
 		)
 		(stroke
@@
 	(wire
 		(pts
-			(xy 300.99 223.52) (xy 304.8 223.52)
+			(xy 295.9642 223.52) (xy 304.8 223.52)
 		)
 		(stroke
@@
 	(wire
 		(pts
+			(xy 391.16 273.05) (xy 391.16 278.13)
+		)
+		(stroke
+			(width 0)
+			(type default)
+		)
+	)
+	(wire
+		(pts
 			(xy 312.42 177.8) (xy 318.77 177.8)
 		)
@@
 	(wire
 		(pts
-			(xy 391.16 267.97) (xy 391.16 278.13)
+			(xy 391.16 267.97) (xy 391.16 273.05)
 		)
 		(stroke
@@
 	(wire
 		(pts
-			(xy 300.99 223.52) (xy 300.99 278.13)
-		)
-		(stroke
-			(width 0)
-			(type default)
-		)
-	)
-	(wire
-		(pts
 			(xy 388.62 233.68) (xy 391.16 233.68)
 		)
@@
 			"AAAAAAAAAAAAAAAAAAAAAAAAAAAAAAAAAAAAAAAAAAAAAAAAAAAAAAAAAAAAAAAAAAAAAAAAAAAA"
 			"AAAAAAAAAAAAAAAAAAAAAAAAAAAAAAAAAAAAAAAAAAAAAAAAAAAAAAAAAAAAAAAAAAAAAAAAAAAA"
+			"AAAAAAAAAAAAAAAAAAAAAAAAAAAAAAAAAAAAAAAAAAAAAAAAAAAAAAAAAAAAAAAAAAAAAAAAAAAA"
+			"AAAAAAAAAAAAAAAAAAAAAAAAAAAAAAAAAAAAAAAAAAAAAAAAAAAAAAAAAAAAAAAAAAAAAAAAAAAA"
+			"AAAAAAAAAAAAAAAAAAAAAAAAAAAAAAAAAAAAAAAAAAAAAAAAAAAAAAAAAAAAAAAAAAAAAAAAAAAA"
+			"AAAAAAAAAAAAAAAAAAAAAAAAAAAAAAAAAAAAAAAAAAAAAAAAAAAAAAAAAAAAAAAAAAAAAAAAAAAA"
+			"AAAAAAAAAAAAAAAAAAAAAAAAAAAAAAAAAAAAAAAAAAAAAAAAAAAAAAAAAAAAAAAAAAAAAAAAAAAA"
+			"AAAAAAAAAAAAAAAAAAAAAAAAAAAAAAAAAAAAAAAAAAAAAAAAAAAAAAAAAAAAAAAAAAAAAAAAAAAA"
+			"AAAAAAAAAAAAAAAAAAAAAAAAAAAAAAAAAAAAAAAAAAAAAAAAAAAAAAAAAAAAAAAAAAAAAAAAAAAA"
+			"AAAAAAAAAAAAAAAAAAAAAAAAAAAAAAAAAAAAAAAAAAAAAAAAAAAAAAAAAAAAAAAAAAAAAAAAAAAA"
+			"AAAAAAAAAAAAAAAAAAAAAAAAAAAAAAAAAAAAAAAAAAAAAAAAAAAAAAAAAAAAAAAAAAAAAAAAAAAA"
+			"AAAAAAAAAAAAAAAAAAAAAAAAAAAAAAAAAAAAAAAAAAAAAAAAAAAAAAAAAAAAAAAAAAAAAAAAAAAA"
+			"AAAAAAAAAAAAAAAAAAAAAAAAAAAAAAAAAAAAAAAAAAAAAAAAAAAAAAAAAAAAAAAAAAAAAAAAAAAA"
+			"AAAAAAAAAAAAAAAAAAAAAAAAAAAAAAAAAAAAAAAAAAAAAAAAAAAAAAAAAAAAAAAAAAAAAAAAAAAA"
+			"AAAAAAAAAAAAAAAAAAAAAAAAAAAAAAAAAAAAAAAAAAAAAAAAAAAAAAAAAAAAAAAAAAAAAAAAAAAA"
+			"AAAAAAAAAAAAAAAAAAAAAAAAAAAAAAAAAAAAAAAAAAAAAAAAAAAAAAAAAAAAAAAAAAAAAAAAAAAA"
+			"AAAAAAAAAAAAAAAAAAAAAAAAAAAAAAAAAAAAAAAAAAAAAAAAAAAAAAAAAAAAAAAAAAAAAAAAAAAA"
+			"AAAAAAAAAAAAAAAAAAAAAAAAAAAAAAAAAAAAAAAAAAAAAAAAAAAAAAAAAAAAAAAAAAAAAAAAAAAA"
+			"AAAAAAAAAAAAAAAAAAAAAAAAAAAAAAAAAAAAAAAAAAAAAAAAAAAAAAAAAAAAAAAAAAAAAAAAAAAA"
+			"AAAAAAAAAAAAAAAAAAAAAAAAAAAAAAAAAAAAAAAAAAAAAAAAAAAAAAAAAAAAAAAAAAAAAAAAAAAA"
 			"AAAAAAAAAAAAAAAAAAAAAAAAAAAAAAAAAA=="
 		)
 	)
+	(hierarchical_label "GND"
+		(shape input)
+		(at 438.15 243.84 0)
+		(effects
+			(font
+				(size 1.27 1.27)
+			)
+			(justify left)
+		)
+	)
 	(hierarchical_label "6p"
 		(shape input)
@@
 		(on_board yes)
 		(dnp no)
-		(fields_autoplaced yes)
 		(property "Reference" "R14M1"
 			(at 393.7 262.8899 0)

Commit message: Integrated in Monitoring board into final pcb
Changed lines of the file:
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@@
 			)
 		)
-		(property "Value" "GND"
+		(property "Value" "GNDM"
 			(at 394.97 290.83 0)
 			(effects

Commit message: Added Transistors for optocouple and relay drive
Changed lines of the file:
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@@
 	)
 	(hierarchical_label "3.3V"
-		(shape input)
+		(shape output)
 		(at 407.67 171.45 90)
 		(effects
@@
 	)
 	(hierarchical_label "5V"
-		(shape input)
+		(shape output)
 		(at 410.21 171.45 90)
 		(effects
