File: BMS-Capstone/BMS_Board.kicad_sch (KiCad schematic)
At the start: 0 parts

Commit message: Added all schematics to main. I was too scared to merge
Parts:
- added C1, C10, C11, C12, C13, C14, C15, C16, C17, C18, C19, C2, C20, C21, C22, C23, C24, C25, C26, C27, C28, C29, C3, C30, C4, C5, C6, C7, C8, C9: C, Capacitor_SMD:C_0805_2012Metric, symbol Device:C
- added IC1, IC2, IC3, IC4, IC5, IC6: MP2643, SamacSys_Parts:MP2639AGRZ, symbol SamacSys_Parts:MP2643
- added L1, L2, L3, L4, L5, L6: L, SamacSys_Parts:MPLAL4020R47 Inductor, symbol Device:L
- added Q1, Q10, Q11, Q12, Q2, Q3, Q4, Q5, Q6, Q7, Q8, Q9: FODM121, SamacSys_Parts:SOP254P675X240-4N, symbol SamacSys_Parts:FODM121
- added R1, R11, R12, R13, R14, R15, R16, R18, R19, R2, R20, R21, R22, R23, R25, R26, R27, R28, R29, R30, R32, R33, R34, R35, R36, R37, R39, R4, R40, R41, R42, R5, R6, R7, R8, R9: R, Resistor_SMD:R_0805_2012Metric, symbol Device:R
- added R10, R17, R24, R3, R31, R38: 0, Resistor_SMD:R_0805_2012Metric, symbol Device:R
Connections:
- new net: IC2.7 (EN), Q4.3 (E), R13.1
- new net: IC3.24 (UBC), R18.1
- new net: IC2.8 (MODE), Q3.3 (E), R14.1
- new net: IC6.8 (MODE), Q11.3 (E), R42.1
- new net: C9.1, R12.1
- new net: C9.2, IC2.4 (SW), L2.1
- new net: C3.2, IC1.17 (CU_FB), R4.2, R5.1
- new net: IC4.22 (LBC), R24.1
- new net: C21.2, IC5.17 (CU_FB), R29.2, R30.1
- new net: C16.2, IC4.17 (CU_FB), R22.2, R23.1
- new net: C29.1, R40.1
- new net: C29.2, IC6.4 (SW), L6.1
- new net: IC3.22 (LBC), R17.1
- new net: C2.2, IC1.4 (SW), L1.1
- new net: IC1.2 (LX), L1.2
- new net: IC4.2 (LX), L4.2
- new net: IC4.24 (UBC), R25.1
- new net: C19.2, IC4.4 (SW), L4.1
- new net: IC4.6 (BST), R26.2
- new net: IC4.7 (EN), Q8.3 (E), R27.1
- new net: IC4.8 (MODE), Q7.3 (E), R28.1
- new net: IC5.7 (EN), Q10.3 (E), R34.1
- new net: IC3.8 (MODE), Q5.3 (E), R21.1
- new net: C26.2, IC6.17 (CU_FB), R36.2, R37.1
- new net: C11.2, IC3.17 (CU_FB), R15.2, R16.1
- new net: C24.2, IC5.4 (SW), L5.1
- new net: IC5.2 (LX), L5.2
- new net: IC3.2 (LX), L3.2
- new net: C14.2, IC3.4 (SW), L3.1
- new net: IC3.6 (BST), R19.2
- new net: IC3.7 (EN), Q6.3 (E), R20.1
- new net: IC1.7 (EN), Q2.3 (E), R6.1
- new net: IC6.22 (LBC), R38.1
- new net: C6.2, IC2.17 (CU_FB), R8.2, R9.1
- new net: IC6.2 (LX), L6.2
- new net: IC2.22 (LBC), R10.1
- new net: C19.1, R26.1
- new net: IC1.22 (LBC), R2.1
- new net: IC1.24 (UBC), R1.1
- new net: IC1.6 (BST), R3.2
- new net: IC1.8 (MODE), Q1.3 (E), R7.1
- new net: IC6.24 (UBC), R39.1
- new net: IC5.22 (LBC), R31.1
- new net: IC6.7 (EN), Q12.3 (E), R41.1
- new net: C14.1, R19.1
- new net: C2.1, R3.1
- new net: IC2.2 (LX), L2.2
- new net: IC2.24 (UBC), R11.1
- new net: IC2.6 (BST), R12.2
- new net: IC5.8 (MODE), Q9.3 (E), R35.1
- new net: C24.1, R33.1
- new net: IC5.6 (BST), R33.2
- new net: IC6.6 (BST), R40.2
- new net: IC5.24 (UBC), R32.1
- new net CELL1+/CELL2-: C10.2, C5.1, C6.1, C7.2, C8.1, IC1.1 (CL), IC2.10 (AGND), IC2.11 (AGND), IC2.12 (AGND), IC2.13 (AGND), IC2.14 (AGND), IC2.15 (AGND), IC2.16 (AGND), IC2.23 (IMAX), IC2.25 (AGND), IC2.26 (AGND), IC2.5 (PGND), Q1.4 (C), Q2.4 (C), R10.2, R11.2, R13.2, R14.2, R9.2
- new net CELL1-: C1.1, C3.1, C4.2, C5.2, IC1.10 (AGND), IC1.11 (AGND), IC1.12 (AGND), IC1.13 (AGND), IC1.14 (AGND), IC1.15 (AGND), IC1.16 (AGND), IC1.23 (IMAX), IC1.25 (AGND), IC1.26 (AGND), IC1.5 (PGND), R1.2, R2.2, R5.2, R6.2, R7.2
- new net CELL2+/CELL3-: C10.1, C11.1, C12.2, C13.1, C15.2, C4.1, IC1.3 (CU), IC2.1 (CL), IC3.10 (AGND), IC3.11 (AGND), IC3.12 (AGND), IC3.13 (AGND), IC3.14 (AGND), IC3.15 (AGND), IC3.16 (AGND), IC3.23 (IMAX), IC3.25 (AGND), IC3.26 (AGND), IC3.5 (PGND), Q3.4 (C), Q4.4 (C), R16.2, R17.2, R18.2, R20.2, R21.2, R4.1
- new net CELL3+/CELL4-: C15.1, C16.1, C17.2, C18.1, C20.2, C7.1, IC2.3 (CU), IC3.1 (CL), IC4.10 (AGND), IC4.11 (AGND), IC4.12 (AGND), IC4.13 (AGND), IC4.14 (AGND), IC4.15 (AGND), IC4.16 (AGND), IC4.23 (IMAX), IC4.25 (AGND), IC4.26 (AGND), IC4.5 (PGND), Q5.4 (C), Q6.4 (C), R23.2, R24.2, R25.2, R27.2, R28.2, R8.1
- new net CELL4+/CELL5-: C12.1, C20.1, C21.1, C22.2, C23.1, C25.2, IC3.3 (CU), IC4.1 (CL), IC5.10 (AGND), IC5.11 (AGND), IC5.12 (AGND), IC5.13 (AGND), IC5.14 (AGND), IC5.15 (AGND), IC5.16 (AGND), IC5.23 (IMAX), IC5.25 (AGND), IC5.26 (AGND), IC5.5 (PGND), Q7.4 (C), Q8.4 (C), R15.1, R30.2, R31.2, R32.2, R34.2, R35.2
- new net CELL5+/CELL6-: C17.1, C25.1, C26.1, C27.2, C28.1, C30.2, IC4.3 (CU), IC5.1 (CL), IC6.10 (AGND), IC6.11 (AGND), IC6.12 (AGND), IC6.13 (AGND), IC6.14 (AGND), IC6.15 (AGND), IC6.16 (AGND), IC6.23 (IMAX), IC6.25 (AGND), IC6.26 (AGND), IC6.5 (PGND), Q10.4 (C), Q9.4 (C), R22.1, R37.2, R38.2, R39.2, R41.2, R42.2
- new net CELL6+/CELL7-: C22.1, C30.1, IC5.3 (CU), IC6.1 (CL), Q11.4 (C), Q12.4 (C), R29.1
- new net CELL7+: C27.1, IC6.3 (CU), R36.1
- new net VCC1: C1.2, IC1.18 (LOGIC), IC1.9 (4V5)
- new net VCC2: C8.2, IC2.18 (LOGIC), IC2.9 (4V5)
- new net VCC3: C13.2, IC3.18 (LOGIC), IC3.9 (4V5)
- new net VCC4: C18.2, IC4.18 (LOGIC), IC4.9 (4V5)
- new net VCC5: C23.2, IC5.18 (LOGIC), IC5.9 (4V5)
- new net VCC6: C28.2, IC6.18 (LOGIC), IC6.9 (4V5)

Commit message: Added connector to balancing schematic
Parts:
- added J4: Conn_01x13_Socket, Connector_PinHeader_2.54mm:PinHeader_1x13_P2.54mm_Vertical, symbol Connector:Conn_01x13_Socket
Connections:
- net CELL1+/CELL2-: now also J4.2 (Pin_2)
- net CELL1-: now also J4.1 (Pin_1)
- net CELL2+/CELL3-: now also J4.3 (Pin_3)
- net CELL3+/CELL4-: now also J4.4 (Pin_4)
- net CELL4+/CELL5-: now also J4.5 (Pin_5)
- net CELL5+/CELL6-: now also J4.6 (Pin_6)
- net CELL6+/CELL7-: now also J4.7 (Pin_7)
- net CELL7+: now also J4.8 (Pin_8)
- new net TH1: J4.10 (Pin_10)
- new net TH2: J4.11 (Pin_11)
- new net TH3: J4.12 (Pin_12)
Other:
- moved on the sheet: C1, C10, C11, C12, C13, C14, C15, C16, C17, C18, C19, C2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

Commit message: relinked footprints
Parts:
- renumbered C16 to C1, C22 to C10, C4 to C11, C27 to C12, C18 to C13, C8 to C14, C13 to C15, C23 to C16, C1 to C17, C28 to C18, C6 to C2, C9 to C20, C14 to C21, C24 to C22, C2 to C23, C29 to C24, C20 to C25, C10 to C26, C15 to C27, C25 to C28, C5 to C29, C11 to C3, C21 to C4, C3 to C5, C26 to C6, C17 to C7, C7 to C8, C12 to C9, IC4 to IC1, IC5 to IC4, IC1 to IC5, L4 to L1, L5 to L4, L1 to L5, Q7 to Q1, Q2 to Q10, Q8 to Q2, Q9 to Q7, Q10 to Q8, Q1 to Q9, R4 to R10, R5 to R11, R36 to R12, R37 to R13, R24 to R14, R10 to R15, R17 to R16, R31 to R17, R2 to R18, R38 to R19, R22 to R2, R25 to R20, R11 to R21, R18 to R22, R32 to R23, R26 to R24, R1 to R25, R39 to R26, R12 to R27, R19 to R28, R33 to R29, R23 to R3, R3 to R30, R40 to R31, R27 to R32, R13 to R33, R20 to R34, R34 to R35, R6 to R36, R41 to R37, R28 to R38, R14 to R39, R8 to R4, R21 to R40, R35 to R41, R7 to R42, R42 to R43, R9 to R5, R15 to R6, R16 to R7, R29 to R8, R30 to R9
