File: BMS-Capstone/BMS_Board.kicad_sch (KiCad schematic)
At the start: 97 parts, among them IC1 MP2643, IC2 MP2643, IC3 MP2643, IC4 MP2643, IC5 MP2643, IC6 MP2643, J4 Conn_01x13_Socket, Q1 FODM121, Q10 FODM121, Q11 FODM121, Q12 FODM121, Q2 FODM121, Q3 FODM121, Q4 FODM121, Q5 FODM121, Q6 FODM121, Q7 FODM121, Q8 FODM121, Q9 FODM121

Commit message: Changed designators for BMS board
Parts:
- renumbered C10_B1 to C10, C11_B1 to C11, C12_B1 to C12, C13_B1 to C13, C14_B1 to C14, C16_B1 to C16, R1_B1 to R1, R2_B1 to R2, R4_B1 to R4, R5_B1 to R5, R6_B1 to R6
Changed lines of the file:
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@@
 		(dnp no)
 		(fields_autoplaced yes)
-		(property "Reference" "R5_B1"
+		(property "Reference" "R5"
 			(at 300.99 80.0099 0)
 			(effects
@@
 			(project "BMS"
 				(path "/f2da9442-ca05-4687-a880-d5cd24c39f1d/3dc06e74-ff57-4ce5-be5c-5d780b9552b6"
-					(reference "R5_B1")
+					(reference "R5")
 					(unit 1)
 				)
@@
 		(dnp no)
 		(fields_autoplaced yes)
-		(property "Reference" "C11_B1"
+		(property "Reference" "C11"
 			(at 307.34 264.1599 0)
 			(effects
@@
 			(project "BMS"
 				(path "/f2da9442-ca05-4687-a880-d5cd24c39f1d/3dc06e74-ff57-4ce5-be5c-5d780b9552b6"
-					(reference "C11_B1")
+					(reference "C11")
 					(unit 1)
 				)
@@
 		(dnp no)
 		(fields_autoplaced yes)
-		(property "Reference" "R6_B1"
+		(property "Reference" "R6"
 			(at 377.19 100.3299 0)
 			(effects
@@
 			(project "BMS"
 				(path "/f2da9442-ca05-4687-a880-d5cd24c39f1d/3dc06e74-ff57-4ce5-be5c-5d780b9552b6"
-					(reference "R6_B1")
+					(reference "R6")
 					(unit 1)
 				)
@@
 		(dnp no)
 		(fields_autoplaced yes)
-		(property "Reference" "C16_B1"
+		(property "Reference" "C16"
 			(at 304.8 356.8699 0)
 			(effects
@@
 			(project "BMS"
 				(path "/f2da9442-ca05-4687-a880-d5cd24c39f1d/3dc06e74-ff57-4ce5-be5c-5d780b9552b6"
-					(reference "C16_B1")
+					(reference "C16")
 					(unit 1)
 				)
@@
 		(dnp no)
 		(fields_autoplaced yes)
-		(property "Reference" "C10_B1"
+		(property "Reference" "C10"
 			(at 375.92 128.2699 0)
 			(effects
@@
 			(project "BMS"
 				(path "/f2da9442-ca05-4687-a880-d5cd24c39f1d/3dc06e74-ff57-4ce5-be5c-5d780b9552b6"
-					(reference "C10_B1")
+					(reference "C10")
 					(unit 1)
 				)
@@
 		(dnp no)
 		(fields_autoplaced yes)
-		(property "Reference" "R1_B1"
+		(property "Reference" "R1"
 			(at 341.63 101.5999 0)
 			(effects
@@
 			(project ""
 				(path "/f2da9442-ca05-4687-a880-d5cd24c39f1d/3dc06e74-ff57-4ce5-be5c-5d780b9552b6"
-					(reference "R1_B1")
+					(reference "R1")
 					(unit 1)
 				)
@@
 		(dnp no)
 		(fields_autoplaced yes)
-		(property "Reference" "C12_B1"
+		(property "Reference" "C12"
 			(at 313.69 229.8699 0)
 			(effects
@@
 			(project "BMS"
 				(path "/f2da9442-ca05-4687-a880-d5cd24c39f1d/3dc06e74-ff57-4ce5-be5c-5d780b9552b6"
-					(reference "C12_B1")
+					(reference "C12")
 					(unit 1)
 				)
@@
 		(dnp no)
 		(fields_autoplaced yes)
-		(property "Reference" "R2_B1"
+		(property "Reference" "R2"
 			(at 328.93 101.5999 0)
 			(effects
@@
 			(project "BMS"
 				(path "/f2da9442-ca05-4687-a880-d5cd24c39f1d/3dc06e74-ff57-4ce5-be5c-5d780b9552b6"
-					(reference "R2_B1")
+					(reference "R2")
 					(unit 1)
 				)
@@
 		(dnp no)
 		(fields_autoplaced yes)
-		(property "Reference" "R4_B1"
+		(property "Reference" "R4"
 			(at 300.99 66.0399 0)
 			(effects
@@
 			(project "BMS"
 				(path "/f2da9442-ca05-4687-a880-d5cd24c39f1d/3dc06e74-ff57-4ce5-be5c-5d780b9552b6"
-					(reference "R4_B1")
+					(reference "R4")
 					(unit 1)
 				)
@@
 		(dnp no)
 		(fields_autoplaced yes)
-		(property "Reference" "C14_B1"
+		(property "Reference" "C14"
 			(at 344.17 204.47 90)
 			(effects
@@
 			(project "BMS"
 				(path "/f2da9442-ca05-4687-a880-d5cd24c39f1d/3dc06e74-ff57-4ce5-be5c-5d780b9552b6"
-					(reference "C14_B1")
+					(reference "C14")
 					(unit 1)
 				)
@@
 		(on_board yes)
 		(dnp no)
-		(property "Reference" "C13_B1"
+		(property "Reference" "C13"
 			(at 313.69 255.778 90)
 			(effects
@@
 			(project "BMS"
 				(path "/f2da9442-ca05-4687-a880-d5cd24c39f1d/3dc06e74-ff57-4ce5-be5c-5d780b9552b6"
-					(reference "C13_B1")
+					(reference "C13")
 					(unit 1)
 				)

Commit message: Final touches
Parts:
- added R43, R44, R45, R46, R47, R48, R49, R50, R51, R52, R53, R54: 200, Resistor_SMD:R_0805_2012Metric, symbol Device:R
- J4: footprint Connector_PinHeader_2.54mm:PinHeader_1x13_P2.54mm_Vertical -> Connector_JST:JST_XH_B13B-XH-A_1x13_P2.50mm_Vertical
Connections:
- net at Q4.1: now also R46.1
- net MCUGND: now reaches Q4.2
- net MCUGND: now also J4.13 (Pin_13), Q1.2, Q10.2, Q11.2, Q12.2, Q2.2, Q3.2, Q5.2, Q6.2, Q7.2, Q8.2, Q9.2
- net at Q11.1: now also R53.1
- net at Q5.1: now also R47.1
- net at Q12.1: now also R54.1
- net at Q1.1: now also R43.1
- net at Q6.1: now also R48.1
- net at Q9.1: now also R51.1
- net at Q8.1: now also R50.1
- net at Q10.1: now also R52.1
- net at Q3.1: now also R45.1
- net RELAY: now reaches J4.9 (Pin_9)
- net at Q2.1: now also R44.1
- net at Q7.1: now also R49.1
- new net 1EN: R44.2
- new net 1MODE: R43.2
- new net 2EN: R46.2
- new net 2MODE: R45.2
- new net 3EN: R48.2
- new net 3MODE: R47.2
- new net 4EN: R50.2
- new net 4MODE: R49.2
- new net 5EN: R52.2
- new net 5MODE: R51.2
- new net 6EN: R54.2
- new net 6MODE: R53.2

Commit message: Added Transistors for optocouple and relay drive
Parts:
- added Q13, Q14, Q15, Q16, Q17, Q18, Q19, Q20, Q21, Q22, Q23, Q24: 2N7002, Package_TO_SOT_SMD:SOT-23, symbol Transistor_FET:2N7002
- added R60, R61, R62, R63, R64, R65, R66, R67, R68, R69, R70, R71: 10k, Resistor_SMD:R_0805_2012Metric, symbol Device:R
- R43, R44, R45, R46, R47, R48, R49, R50, R51, R52, R53, R54: value 200 -> 720
Connections:
- net 1EN: now also Q14.1 (G), R61.1; no longer R44.2
- net 1MODE: now also Q13.1 (G), R60.1; no longer R43.2
- net 2EN: now also Q16.1 (G), R63.1; no longer R46.2
- net 2MODE: now also Q15.1 (G), R62.1; no longer R45.2
- net 3EN: now also Q18.1 (G), R65.1; no longer R48.2
- net 3MODE: now also Q17.1 (G), R64.1; no longer R47.2
- net 4EN: now also Q20.1 (G), R67.1; no longer R50.2
- net 4MODE: now also Q19.1 (G), R66.1; no longer R49.2
- net 5EN: now also Q22.1 (G), R69.1; no longer R52.2
- net 5MODE: now also Q21.1 (G), R68.1; no longer R51.2
- net 6EN: now also Q24.1 (G), R71.1; no longer R54.2
- net 6MODE: now also Q23.1 (G), R70.1; no longer R53.2
- net MCUGND: now also Q13.2 (S), Q14.2 (S), Q15.2 (S), Q16.2 (S), Q17.2 (S), Q18.2 (S), Q19.2 (S), Q20.2 (S), Q21.2 (S), Q22.2 (S), Q23.2 (S), Q24.2 (S), R60.2, R61.2, R62.2, R63.2, R64.2, R65.2, R66.2, R67.2, R68.2, R69.2, R70.2, R71.2; no longer Q1.2, Q10.2, Q11.2, Q12.2, Q2.2, Q3.2, Q4.2, Q5.2, Q6.2, Q7.2, Q8.2, Q9.2
- new net: Q16.3 (D), Q4.2
- new net: Q11.2, Q23.3 (D)
- new net: Q19.3 (D), Q7.2
- new net: Q17.3 (D), Q5.2
- new net: Q12.2, Q24.3 (D)
- new net: Q21.3 (D), Q9.2
- new net: Q15.3 (D), Q3.2
- new net: Q10.2, Q22.3 (D)
- new net: Q1.2, Q13.3 (D)
- new net: Q18.3 (D), Q6.2
- new net: Q20.3 (D), Q8.2
- new net: Q14.3 (D), Q2.2
- new net 5v: R43.2, R44.2, R45.2, R46.2, R47.2, R48.2, R49.2, R50.2, R51.2, R52.2, R53.2, R54.2
Other:
- moved on the sheet: J4

Commit message: Generated BOM
Parts:
- C1, C13, C18, C23, C28, C8: value C -> 1u
- C10, C12, C15, C17, C20, C22, C25, C27, C30, C4, C5, C7: value C -> 22u
- C11, C16, C21, C26, C3, C6: value C -> 1n
- C14, C19, C2, C29, C9: value C -> 100n
- C24: value C -> 100nF
- L1, L2, L3, L4, L5, L6: value L -> 1uH
- R1, R11, R18, R25, R32, R39: value R -> 120k
- R10, R17, R24, R31, R38: value 0 -> 150k
- R12, R19, R26, R33, R40: value R -> 0
- R13, R14, R20, R21, R27, R28, R34, R35, R41, R42, R6, R7: value R -> 10k
- R15, R22, R29, R36, R4, R8: value R -> 2M
- R16, R23, R30, R37, R5, R9: value R -> 330k
- R2: value R -> 150k
