File: BMS-Capstone/Battery_Pack.kicad_sch (KiCad schematic)
At the start: 0 parts

Commit message: Added main Schematic to branch and linked components to PCB
Parts:
- added BT1, BT2, BT3, BT4, BT5, BT6, BT7: Battery_Cell, cell:keystone 254 18650, symbol Device:Battery_Cell
- added F1: Fuse, Fuse:Fuseholder_Blade_Mini_Keystone_3568, symbol Device:Fuse
- added J1: Conn_01x02_Socket, Connector_PinHeader_2.54mm:PinHeader_1x02_P2.54mm_Vertical, symbol Connector:Conn_01x02_Socket
- added J2: Conn_01x02_Socket, cell:XT60, symbol Connector:Conn_01x02_Socket
- added J3: Conn_01x13_Socket, Connector_PinHeader_2.54mm:PinHeader_1x13_P2.54mm_Vertical, symbol Connector:Conn_01x13_Socket
- added K1: J107F1CS203VDC.80, cell:3_3v relay, symbol Relay:DIPxx-1Cxx-51x
- added R1: R, Resistor_SMD:R_1210_3225Metric, symbol Device:R
- added TH1, TH2, TH3: Thermistor, Resistor_THT:R_Axial_DIN0204_L3.6mm_D1.6mm_P2.54mm_Vertical, symbol Device:Thermistor
Connections:
- new net: F1.1, J1.2 (Pin_2), R1.2
- new net: J2.1 (Pin_1), K1.14
- new net: J3.9 (Pin_9), K1.6
- new net 1+: BT1.1 (+), BT2.2 (-), J3.2 (Pin_2)
- new net 1-: BT1.2 (-), J1.1 (Pin_1), J3.1 (Pin_1), R1.1
- new net 2+: BT2.1 (+), BT3.2 (-), J3.3 (Pin_3)
- new net 3+: BT3.1 (+), BT4.2 (-), J3.4 (Pin_4)
- new net 4+: BT4.1 (+), BT5.2 (-), J3.5 (Pin_5)
- new net 5+: BT5.1 (+), BT6.2 (-), J3.6 (Pin_6)
- new net 6+: BT6.1 (+), BT7.2 (-), J3.7 (Pin_7)
- new net 7+: BT7.1 (+), J3.8 (Pin_8), K1.7, K1.8
- new net GND: F1.2, J2.2 (Pin_2)
- new net MCUGND: J3.13 (Pin_13), K1.2, TH1.2, TH2.2, TH3.2
- new net TH1: J3.10 (Pin_10), TH1.1
- new net TH2: J3.11 (Pin_11), TH2.1
- new net TH3: J3.12 (Pin_12), TH3.1

Commit message: relinked footprints
Parts:
- renumbered BT7 to BT1, BT6 to BT2, BT5 to BT3, BT3 to BT5, BT2 to BT6, BT1 to BT7, J3 to J1, J1 to J3, TH3 to TH1, TH1 to TH3
Changed lines of the file:
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@@
 		(dnp no)
 		(fields_autoplaced yes)
-		(property "Reference" "BT1"
+		(property "Reference" "BT7"
 			(at 138.43 150.5584 0)
 			(effects
@@
 			(project ""
 				(path "/f2da9442-ca05-4687-a880-d5cd24c39f1d/cf34981b-cbae-442d-9f72-9ae4895e9d63"
-					(reference "BT1")
+					(reference "BT7")
 					(unit 1)
 				)
@@
 		(dnp no)
 		(fields_autoplaced yes)
-		(property "Reference" "BT6"
+		(property "Reference" "BT2"
 			(at 138.43 88.3284 0)
 			(effects
@@
 			(project "BMS"
 				(path "/f2da9442-ca05-4687-a880-d5cd24c39f1d/cf34981b-cbae-442d-9f72-9ae4895e9d63"
-					(reference "BT6")
+					(reference "BT2")
 					(unit 1)
 				)
@@
 		(dnp no)
 		(fields_autoplaced yes)
-		(property "Reference" "BT5"
+		(property "Reference" "BT3"
 			(at 138.43 101.0284 0)
 			(effects
@@
 			(project "BMS"
 				(path "/f2da9442-ca05-4687-a880-d5cd24c39f1d/cf34981b-cbae-442d-9f72-9ae4895e9d63"
-					(reference "BT5")
+					(reference "BT3")
 					(unit 1)
 				)
@@
 		(dnp no)
 		(fields_autoplaced yes)
-		(property "Reference" "BT3"
+		(property "Reference" "BT5"
 			(at 138.43 126.4284 0)
 			(effects
@@
 			(project "BMS"
 				(path "/f2da9442-ca05-4687-a880-d5cd24c39f1d/cf34981b-cbae-442d-9f72-9ae4895e9d63"
-					(reference "BT3")
+					(reference "BT5")
 					(unit 1)
 				)
@@
 		(dnp no)
 		(fields_autoplaced yes)
-		(property "Reference" "#PWR01"
+		(property "Reference" "#PWR03"
 			(at 134.62 185.42 0)
 			(effects
@@
 			(project ""
 				(path "/f2da9442-ca05-4687-a880-d5cd24c39f1d/cf34981b-cbae-442d-9f72-9ae4895e9d63"
-					(reference "#PWR01")
+					(reference "#PWR03")
 					(unit 1)
 				)
@@
 		(dnp no)
 		(fields_autoplaced yes)
-		(property "Reference" "#PWR02"
+		(property "Reference" "#PWR05"
 			(at 157.48 91.44 0)
 			(effects
@@
 			(project "BMS"
 				(path "/f2da9442-ca05-4687-a880-d5cd24c39f1d/cf34981b-cbae-442d-9f72-9ae4895e9d63"
-					(reference "#PWR02")
+					(reference "#PWR05")
 					(unit 1)
 				)
@@
 		(dnp no)
 		(fields_autoplaced yes)
-		(property "Reference" "#PWR04"
+		(property "Reference" "#PWR07"
 			(at 162.56 153.67 0)
 			(effects
@@
 			(project "BMS"
 				(path "/f2da9442-ca05-4687-a880-d5cd24c39f1d/cf34981b-cbae-442d-9f72-9ae4895e9d63"
-					(reference "#PWR04")
+					(reference "#PWR07")
 					(unit 1)
 				)
@@
 		(dnp no)
 		(fields_autoplaced yes)
-		(property "Reference" "TH3"
+		(property "Reference" "TH1"
 			(at 161.29 78.7399 0)
 			(effects
@@
 			(project "BMS"
 				(path "/f2da9442-ca05-4687-a880-d5cd24c39f1d/cf34981b-cbae-442d-9f72-9ae4895e9d63"
-					(reference "TH3")
+					(reference "TH1")
 					(unit 1)
 				)
@@
 		(dnp no)
 		(fields_autoplaced yes)
-		(property "Reference" "#PWR07"
+		(property "Reference" "#PWR01"
 			(at 72.39 102.87 0)
 			(effects
@@
 			(project ""
 				(path "/f2da9442-ca05-4687-a880-d5cd24c39f1d/cf34981b-cbae-442d-9f72-9ae4895e9d63"
-					(reference "#PWR07")
+					(reference "#PWR01")
 					(unit 1)
 				)
@@
 		(dnp no)
 		(fields_autoplaced yes)
-		(property "Reference" "J3"
+		(property "Reference" "J1"
 			(at 51.435 88.9 0)
 			(effects
@@
 			(project ""
 				(path "/f2da9442-ca05-4687-a880-d5cd24c39f1d/cf34981b-cbae-442d-9f72-9ae4895e9d63"
-					(reference "J3")
+					(reference "J1")
 					(unit 1)
 				)
@@
 		(dnp no)
 		(fields_autoplaced yes)
-		(property "Reference" "#PWR03"
+		(property "Reference" "#PWR06"
 			(at 157.48 125.73 0)
 			(effects
@@
 			(project "BMS"
 				(path "/f2da9442-ca05-4687-a880-d5cd24c39f1d/cf34981b-cbae-442d-9f72-9ae4895e9d63"
-					(reference "#PWR03")
+					(reference "#PWR06")
 					(unit 1)
 				)
@@
 		(dnp no)
 		(fields_autoplaced yes)
-		(property "Reference" "#PWR06"
+		(property "Reference" "#PWR04"
 			(at 139.7 44.45 0)
 			(effects
@@
 			(project "BMS"
 				(path "/f2da9442-ca05-4687-a880-d5cd24c39f1d/cf34981b-cbae-442d-9f72-9ae4895e9d63"
-					(reference "#PWR06")
+					(reference "#PWR04")
 					(unit 1)
 				)
@@
 		(dnp no)
 		(fields_autoplaced yes)
-		(property "Reference" "#PWR08"
+		(property "Reference" "#PWR02"
 			(at 124.46 66.04 0)
 			(effects
@@
 			(project "BMS"
 				(path "/f2da9442-ca05-4687-a880-d5cd24c39f1d/cf34981b-cbae-442d-9f72-9ae4895e9d63"
-					(reference "#PWR08")
+					(reference "#PWR02")
 					(unit 1)
 				)
@@
 		(dnp no)
 		(fields_autoplaced yes)
-		(property "Reference" "BT2"
+		(property "Reference" "BT6"
 			(at 138.43 139.1284 0)
 			(effects
@@
 			(project "BMS"
 				(path "/f2da9442-ca05-4687-a880-d5cd24c39f1d/cf34981b-cbae-442d-9f72-9ae4895e9d63"
-					(reference "BT2")
+					(reference "BT6")
 					(unit 1)
 				)
@@
 		(dnp no)
 		(fields_autoplaced yes)
-		(property "Reference" "J1"
+		(property "Reference" "J3"
 			(at 151.13 162.5599 0)
 			(effects
@@
 			(project ""
 				(path "/f2da9442-ca05-4687-a880-d5cd24c39f1d/cf34981b-cbae-442d-9f72-9ae4895e9d63"
-					(reference "J1")
+					(reference "J3")
 					(unit 1)
 				)
@@
 		(dnp no)
 		(fields_autoplaced yes)
-		(property "Reference" "BT7"
+		(property "Reference" "BT1"
 			(at 138.43 74.3584 0)
 			(effects
@@
 			(project "BMS"
 				(path "/f2da9442-ca05-4687-a880-d5cd24c39f1d/cf34981b-cbae-442d-9f72-9ae4895e9d63"
-					(reference "BT7")
+					(reference "BT1")
 					(unit 1)
 				)
@@
 		(dnp no)
 		(fields_autoplaced yes)
-		(property "Reference" "TH1"
+		(property "Reference" "TH3"
 			(at 166.37 140.9699 0)
 			(effects
@@
 			(project ""
 				(path "/f2da9442-ca05-4687-a880-d5cd24c39f1d/cf34981b-cbae-442d-9f72-9ae4895e9d63"
-					(reference "TH1")
-					(unit 1)
-				)
+					(reference "TH3")
+					(unit 1)
+				)
