File: BMS-Capstone/Teensy_4.0.kicad_sch (KiCad schematic)
At the start: 1 part, among them U1 Teensy4.0

Commit message: Final touches
Parts:
- added R55, R56, R57: 10K, Resistor_SMD:R_0805_2012Metric, symbol Device:R
- added R58, R59: 0, Resistor_SMD:R_0805_2012Metric, symbol Device:R
Connections:
- net 3V3: now also R55.2, R56.2, R57.2, R58.2, R59.1; no longer U1.33 (VIN)
- net 6MODE: now reaches U1.10 (8_TX2_IN1)
- net INT: now reaches U1.11 (9_OUT1C)
- net at U1.16 (3V3): now also R58.1
- net RELAY: now reaches U1.2 (0_RX1_CRX2_CS1)
- net TH1: now reaches U1.21 (14_A0_TX3_SPDIF_OUT)
- net TH1: now also R55.1
- net TH2: now reaches U1.22 (15_A1_RX3_SPDIF_IN)
- net TH2: now also R56.1
- net TH3: now reaches U1.23 (16_A2_RX4_SCL1)
- net TH3: now also R57.1
- net 5MODE: now reaches U1.27 (20_A6_TX5_LRCLK1)
- net 5EN: now reaches U1.28 (21_A7_RX5_BCLK1)
- net 4MODE: now reaches U1.29 (22_A8_CTX1)
- net 1MODE: now reaches U1.3 (1_TX1_CTX2_MISO1)
- net 4EN: now reaches U1.30 (23_A9_CRX1_MCLK1)
- net 1EN: now reaches U1.4 (2_OUT2)
- net 2MODE: now reaches U1.5 (3_LRCLK2)
- net 2EN: now reaches U1.6 (4_BCLK2)
- net 3MODE: now reaches U1.7 (5_IN2)
- net 3EN: now reaches U1.8 (6_OUT1D)
- net 6EN: now reaches U1.9 (7_RX2_OUT1A)
- new net: R59.2, U1.33 (VIN)
